File: EC1834-XT-IDE.kicad_pcb (KiCad board)
At the start: 2 copper layers, 114.3 x 109.9 mm, 46 parts, among them J1 CONN_3, J2 CONN_3, J3 CONN_2, J4 CONN_2, J5 INTERRUPT, P6 CONN_1, P7 CONN_1, SW1 I/O ADDR, SW2 ROM OPT, U1 74LS573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

Commit message: Moved some tracks to move drill holes for new slot sheet position in EC1834
Parts:
- moved P6 12.1 mm to (186.7, 140.3)
- moved P7 12.1 mm to (186.7, 83.8)
Connections:
- SW1 pad 8: *CARDSEL -> (no net)
Routing:
- net *CARDSEL: track 88.1 -> 0.00 mm
- net GND: track 33.3 -> 23.8 mm
- net D7: track 247.5 -> 241.1 mm
- net RESDRV: track 113.3 -> 107.6 mm
- net D6: track 174.4 -> 169.5 mm
- net D5: track 174.2 -> 169.6 mm
- net *CS_IDE: track 215.0 -> 212.4 mm
- net D4: track 172.8 -> 170.3 mm
- net D3: track 176.4 -> 174.2 mm
- net D2: track 176.4 -> 174.6 mm
- net D1: track 176.4 -> 174.9 mm
- net D0: track 176.4 -> 175.7 mm
Other:
- outline, holes or cut-outs redrawn
- board text added: "(c)2022 M. Goegel"
- board text added: "EC1834-XT-IDE based on rev 04 (c) 2017 The Glitch Works https://github.com/mgoegel/EC1834-XT-IDE"
- board text added: "NC"
- board text removed: "XT-IDE rev 04 (c) 2017 The Glitch Works http://www.glitchwrks.com/xt-ide"
- board text removed: "XT8"

Commit message: Moved some ICs Prepared new arrangement
Parts:
- moved J4 45.4 mm to (59.1, 98.4)
- moved IDE1 39.8 mm to (47.6, 101.6)
- moved RP1 37.9 mm to (60.3, 118.7)
- moved SW1 37.9 mm to (47.6, 112.4)
- moved C12 36.7 mm to (52.7, 138.4), turned to 180 degrees
Other:
- board size 114.3 x 109.9 mm -> 153.7 x 109.9 mm
- board text added: "Max board height"
