File: KiCad/EC1834-XT-IDE.sch (KiCad schematic (older format))
At the start: 45 parts, among them J1 CONN_3, J2 CONN_3, J3 CONN_2, J4 CONN_2, J5 INTERRUPT, P6 CONN_1, P7 CONN_1, SW1 I/O ADDR, SW2 ROM OPT, U1 74LS573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

Commit message: Reorganzied KiCad project Completed PCB, added some configuration notes on PCB
Parts:
- removed BUS1: BUSPC, edge_connectors:ISA-8BIT-XT-IDE, symbol XT-IDE-rescue:BUSPC
- removed TP1, TP2, TP3: CONN_1, testpoints:TH_TESTPOINT, symbol XT-IDE-rescue:CONN_1
- BUS1: footprint Connector_DIN:DIN41612_C_2x32_Male_Horizontal_THT -> Connector_DIN:DIN41612_C_3x32_Male_Horizontal_THT; symbol EC1834-ISA:BUS_EC1834_8Bit -> EC1834-XT-IDE-rescue:BUS_EC1834_8Bit-EC1834-ISA
Connections:
- net labels removed: *CARDSEL, *CARDSEL_SWITCHED
- wire segments 444 -> 438
- no-connect marks 23 -> 25
Other:
- note added: "No Slot 8 Support mod supported on EC1834"
- note added: "ROM Address Notes:\nFor full 32K device (28C256) set S1 3,4,5,6 ON\nFor 8K device (28C64B) set S1 5,6 OFF\nS1 3,4 become address switches"
- note added: "Switch Settings\n1-4 ROM Address (OFF == 1)\n5 A14 Enable (OFF == enabled)\n6 A13 (OFF == enabled)\n7 ROM Enable (OFF == enabled)\n8 Write Enable (OFF == enabled)"
- note removed: "Card Select (XT Slot 8 Support)"
- note removed: "For use with Slot 8 Support mod"
- note removed: "ROM Address Notes:\nFor full 32K device (28C256) set S1 3,4,5,6 OFF\nFor 8K device (28C64B) set S1 5,6 ON\nS1 3,4 become address switches"
- note removed: "Slot 8 Suppor Test Points"
- note removed: "Switch Settings\n1-4 ROM Address (ON == 1)\n5 A14 Enable (ON == enabled)\n6 A13 (ON == enabled)\n7 ROM Enable (ON == enabled)\n8 Write Enable (ON == enabled)"

Commit message: Updated schema revision Updated gerber files Added default BIOS
Parts:
- added IDE2: CONN_22X2, Connector_PinSocket_2.00mm:PinSocket_2x22_P2.00mm_Horizontal, symbol Connector_Generic:Conn_02x22_Odd_Even
Connections:
- net labels added: DMARQ.2, IOCS16.2, PDIAG.2
- wire segments 438 -> 484
- no-connect marks 25 -> 28
Other:
- note added: "IDE/CF POWER SUPPLY \nOPTION JUMPER"
- note added: "ROM Address Notes:\nFor full 32K device (28C256) set S1 3,4,5,6 OFF\nFor 8K device (28C64B) set S1 5,6 ON\nS1 3,4 become address switches"
- note added: "Switch Settings\n1-4 ROM Address (ON == 1)\n5 A14 Enable (ON == enabled)\n6 A13 (ON == enabled)\n7 ROM Enable (ON == enabled)\n8 Write Enable (ON == enabled)"
- note removed: "IDE/CF POWER SUPPLY OPTION JUMPER"
- note removed: "ROM Address Notes:\nFor full 32K device (28C256) set S1 3,4,5,6 ON\nFor 8K device (28C64B) set S1 5,6 OFF\nS1 3,4 become address switches"
- note removed: "Switch Settings\n1-4 ROM Address (OFF == 1)\n5 A14 Enable (OFF == enabled)\n6 A13 (OFF == enabled)\n7 ROM Enable (OFF == enabled)\n8 Write Enable (OFF == enabled)"
- moved on the sheet: J4
